File: BCN3D++.sch (EAGLE design)
At the start: 87 parts, among them IC2 FT232RL, Q2 IRLS3034

Commit message: Main Board almost ready
5V rail to ICSP and some headers left to connect
Parts:
- removed GND20: PTR1TP12SQ, testpad:PTR1TP12SQ
Connections:
- removed net N$128: ATMEGA2560.(OC0B)_PG5
- new net 11111: ATMEGA2560.(OC2A/PCINT4)_PB4
- net +24V: now also 24V.TP
- net +5V: no longer 24V.TP
- net GND: no longer GND20.TP
- net PWM_HOTBED: now also ATMEGA2560.(OC0B)_PG5; no longer ATMEGA2560.(OC2A/PCINT4)_PB4
Other:
- moved on the sheet: +5V, R16
Changed lines of the file:
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@@
 <part name="+5V" library="testpad" deviceset="PTR1" device="TP12SQ" value=""/>
 <part name="GND52" library="supply1" deviceset="GND" device=""/>
-<part name="P+52" library="supply1" deviceset="+5V" device="" value="+24V"/>
-<part name="P+53" library="supply1" deviceset="+5V" device=""/>
 <part name="FID1" library="adafruit" deviceset="FIDUCIAL" device=""/>
 <part name="U$1" library="SAV MK-I" deviceset="SANGUINOLOLU_PLATED-SCREW" device=""/>
@@
 <part name="FID3" library="adafruit" deviceset="FIDUCIAL" device=""/>
 <part name="+24V" library="SparkFun-Connectors" deviceset="M02" device="5MM" value="control"/>
-<part name="GND20" library="testpad" deviceset="PTR1" device="TP12SQ" value="PTR1TP12SQ"/>
-<part name="GND16" library="supply1" deviceset="GND" device=""/>
 <part name="SD" library="MarcEagleParts" deviceset="M06" device="SIP"/>
 <part name="ENDSTOPS" library="MarcEagleParts" deviceset="PINCONNECTOR-7X3" device=""/>
@@
 <instance part="P+27" gate="1" x="251.46" y="363.22"/>
 <instance part="GND27" gate="1" x="256.54" y="281.94"/>
-<instance part="R16" gate="G$1" x="314.96" y="213.36" rot="R180"/>
+<instance part="R16" gate="G$1" x="312.42" y="213.36" rot="R180"/>
 <instance part="R17" gate="G$1" x="320.04" y="208.28" rot="R270"/>
 <instance part="D3" gate="G$1" x="320.04" y="228.6" rot="R90"/>
@@
 <instance part="GND" gate="G$1" x="162.56" y="347.98" rot="R180"/>
 <instance part="24V" gate="G$1" x="170.18" y="347.98"/>
-<instance part="+5V" gate="G$1" x="182.88" y="347.98"/>
+<instance part="+5V" gate="G$1" x="177.8" y="347.98"/>
 <instance part="GND52" gate="1" x="162.56" y="342.9"/>
-<instance part="P+52" gate="1" x="170.18" y="355.6"/>
-<instance part="P+53" gate="1" x="182.88" y="355.6"/>
 <instance part="FID1" gate="G$1" x="-55.88" y="83.82"/>
 <instance part="U$1" gate="G$1" x="215.9" y="358.14"/>
@@
 <instance part="FID3" gate="G$1" x="-44.196" y="83.82"/>
 <instance part="+24V" gate="G$1" x="40.64" y="294.64"/>
-<instance part="GND20" gate="G$1" x="175.26" y="347.98" rot="R180"/>
-<instance part="GND16" gate="1" x="175.26" y="342.9"/>
 <instance part="SD" gate="G$1" x="165.1" y="284.48"/>
 <instance part="ENDSTOPS" gate="-1" x="261.62" y="353.06" rot="R270"/>
@@
 <pinref part="FANS" gate="-3" pin="2"/>
 <pinref part="FANS" gate="-4" pin="2"/>
-</segment>
-<segment>
-<pinref part="GND20" gate="G$1" pin="TP"/>
-<pinref part="GND16" gate="1" pin="GND"/>
 </segment>
 <segment>
@@
 </segment>
 <segment>
-<pinref part="+5V" gate="G$1" pin="TP"/>
-<pinref part="P+53" gate="1" pin="+5V"/>
-<wire x1="182.88" y1="350.52" x2="182.88" y2="353.06" width="0.1524" layer="91"/>
-</segment>
-<segment>
-<pinref part="24V" gate="G$1" pin="TP"/>
-<pinref part="P+52" gate="1" pin="+5V"/>
-<wire x1="170.18" y1="350.52" x2="170.18" y2="353.06" width="0.1524" layer="91"/>
-</segment>
-<segment>
 <pinref part="X0-AXIS" gate="G$1" pin="3"/>
 <wire x1="297.18" y1="335.28" x2="307.34" y2="335.28" width="0.1524" layer="91"/>
@@
 <pinref part="FANS" gate="-4" pin="1"/>
 </segment>
+<segment>
+<pinref part="+5V" gate="G$1" pin="TP"/>
+<wire x1="177.8" y1="350.52" x2="177.8" y2="355.6" width="0.1524" layer="91"/>
+<wire x1="177.8" y1="355.6" x2="182.88" y2="355.6" width="0.1524" layer="91"/>
+<label x="177.8" y="353.06" size="1.778" layer="95"/>
+</segment>
 </net>
 <net name="N$2" class="0">
@@
 <pinref part="R17" gate="G$1" pin="1"/>
 <pinref part="Q2" gate="G$1" pin="G"/>
-<wire x1="320.04" y1="213.36" x2="327.66" y2="213.36" width="0.1524" layer="91"/>
-<junction x="320.04" y="213.36"/>
+<wire x1="317.5" y1="213.36" x2="327.66" y2="213.36" width="0.1524" layer="91"/>
+<junction x="317.5" y="213.36"/>
+<wire x1="317.5" y1="213.36" x2="320.04" y2="213.36" width="0.1524" layer="91"/>
 </segment>
 </net>
@@
 <segment>
 <pinref part="R16" gate="G$1" pin="2"/>
-<wire x1="309.88" y1="213.36" x2="289.56" y2="213.36" width="0.1524" layer="91"/>
+<wire x1="307.34" y1="213.36" x2="289.56" y2="213.36" width="0.1524" layer="91"/>
 <label x="289.56" y="213.36" size="1.778" layer="95"/>
 </segment>
 <segment>
-<pinref part="ATMEGA2560" gate="A" pin="(OC2A/PCINT4)_PB4"/>
-<wire x1="12.7" y1="182.88" x2="-5.08" y2="182.88" width="0.1524" layer="91"/>
-<label x="-2.54" y="182.88" size="1.778" layer="95"/>
+<pinref part="ATMEGA2560" gate="A" pin="(OC0B)_PG5"/>
+<wire x1="104.14" y1="200.66" x2="124.46" y2="200.66" width="0.1524" layer="91"/>
+<label x="106.68" y="200.66" size="1.778" layer="95"/>
 </segment>
 </net>
@@
 <pinref part="ATMEGA2560" gate="A" pin="PC0_(A8)"/>
 <wire x1="12.7" y1="170.18" x2="-5.08" y2="170.18" width="0.1524" layer="91"/>
-<label x="-2.54" y="170.18" size="1.778" layer="95"/>
 </segment>
 </net>
@@
 <pinref part="ATMEGA2560" gate="A" pin="PC1_(A9)"/>
 <wire x1="12.7" y1="167.64" x2="-5.08" y2="167.64" width="0.1524" layer="91"/>
-<label x="-2.54" y="167.64" size="1.778" layer="95"/>
 </segment>
 </net>
@@
 <pinref part="ATMEGA2560" gate="A" pin="PC2_(A10)"/>
 <wire x1="12.7" y1="165.1" x2="-5.08" y2="165.1" width="0.1524" layer="91"/>
-<label x="-2.54" y="165.1" size="1.778" layer="95"/>
 </segment>
 </net>
@@
 <pinref part="ATMEGA2560" gate="A" pin="PC3_(A11)"/>
 <wire x1="12.7" y1="162.56" x2="-5.08" y2="162.56" width="0.1524" layer="91"/>
-<label x="-2.54" y="162.56" size="1.778" layer="95"/>
 </segment>
 </net>
@@
 <pinref part="ATMEGA2560" gate="A" pin="PC4_(A12)"/>
 <wire x1="12.7" y1="160.02" x2="-5.08" y2="160.02" width="0.1524" layer="91"/>
-<label x="-2.54" y="160.02" size="1.778" layer="95"/>
 </segment>
 </net>
@@
 <pinref part="ATMEGA2560" gate="A" pin="PC5_(A13)"/>
 <wire x1="12.7" y1="157.48" x2="-5.08" y2="157.48" width="0.1524" layer="91"/>
-<label x="-2.54" y="157.48" size="1.778" layer="95"/>
 </segment>
 </net>
@@
 <pinref part="ATMEGA2560" gate="A" pin="PC6_(A14)"/>
 <wire x1="12.7" y1="154.94" x2="-5.08" y2="154.94" width="0.1524" layer="91"/>
-<label x="-2.54" y="154.94" size="1.778" layer="95"/>
 </segment>
 </net>
@@
 <pinref part="ATMEGA2560" gate="A" pin="PC7_(A15)"/>
 <wire x1="12.7" y1="152.4" x2="-5.08" y2="152.4" width="0.1524" layer="91"/>
-<label x="-2.54" y="152.4" size="1.778" layer="95"/>
 </segment>
 </net>
@@
 <pinref part="ATMEGA2560" gate="A" pin="(XCK1)_PD5"/>
 <wire x1="12.7" y1="134.62" x2="-5.08" y2="134.62" width="0.1524" layer="91"/>
-<label x="-2.54" y="134.62" size="1.778" layer="95"/>
 </segment>
 </net>
@@
 <pinref part="ATMEGA2560" gate="A" pin="(T1)_PD6"/>
 <wire x1="12.7" y1="132.08" x2="-5.08" y2="132.08" width="0.1524" layer="91"/>
-<label x="-2.54" y="132.08" size="1.778" layer="95"/>
 </segment>
 </net>
@@
 <pinref part="ATMEGA2560" gate="A" pin="(T0)_PD7"/>
 <wire x1="12.7" y1="129.54" x2="-5.08" y2="129.54" width="0.1524" layer="91"/>
-<label x="-2.54" y="129.54" size="1.778" layer="95"/>
 </segment>
 </net>
@@
 <pinref part="ATMEGA2560" gate="A" pin="(TOSC1)_PG4"/>
 <wire x1="104.14" y1="203.2" x2="124.46" y2="203.2" width="0.1524" layer="91"/>
-</segment>
-</net>
-<net name="N$128" class="0">
-<segment>
-<pinref part="ATMEGA2560" gate="A" pin="(OC0B)_PG5"/>
-<wire x1="104.14" y1="200.66" x2="124.46" y2="200.66" width="0.1524" layer="91"/>
 </segment>
 </net>
@@
 <label x="347.98" y="154.94" size="1.778" layer="95"/>
 </segment>
+<segment>
+<pinref part="24V" gate="G$1" pin="TP"/>
+<wire x1="170.18" y1="350.52" x2="170.18" y2="355.6" width="0.1524" layer="91"/>
+<wire x1="170.18" y1="355.6" x2="175.26" y2="355.6" width="0.1524" layer="91"/>
+<label x="170.18" y="353.06" size="1.778" layer="95"/>
+</segment>
 </net>
 <net name="N$161" class="0">
@@
 </segment>
 </net>
+<net name="11111" class="0">
+<segment>
+<pinref part="ATMEGA2560" gate="A" pin="(OC2A/PCINT4)_PB4"/>
+<wire x1="12.7" y1="182.88" x2="-5.08" y2="182.88" width="0.1524" layer="91"/>
+</segment>
+</net>
