File: Heated Bed/BCNmk2.brd (EAGLE design)
At the start: 297 x 210 mm, 16 parts

Commit message: The new REV_B has been shipped to production
New MainBoard Design, new Stepper drivers and new Extruder Board.
We also added many new components and configurations
Parts:
- removed E$1, E$2, E$3, E$4: (no value), holes:3,2-PAD
- added 100K-NTC: (no value), resistor:R0805
- added NTC: 100K, SparkFun-Connectors:1X02
- E$5: device MarcEagleParts:BCN3D_LOGO_HUGE -> MarcEagleParts:BCN3D_PRINTER_HUGE
- moved E$10 26.0 mm to (258.0, 143.0)
- moved E$11 26.0 mm to (258.0, 40.0)
- moved E$8 26.0 mm to (258.0, 65.0)
- moved E$9 26.0 mm to (258.0, 168.0)
- moved E$12 25.0 mm to (10.0, 40.0)
- moved E$6 25.0 mm to (10.0, 65.0)
- moved E$13 24.0 mm to (11.0, 145.0)
- moved E$7 24.0 mm to (11.0, 170.0)
- moved E$5 12.9 mm to (91.0, 143.0)
Routing:
- net S$5: track 1866.9 -> 0.00 mm
- net S$4: track 1869.7 -> 3549.7 mm
- net S$41: track 2060.4 -> 1306.8 mm
- net GND: track 0.00 -> 369.5 mm, vias 0 -> 21
- net S$3: track 355.2 -> 0.00 mm
- net S$2: track 350.9 -> 0.00 mm
- net +24: track 0.00 -> 267.4 mm, vias 0 -> 18
- net S$40: track 1866.9 -> 2114.6 mm
- net -NTC: track 0.00 -> 145.4 mm, vias 0 -> 1
- net +NTC: track 0.00 -> 144.6 mm, vias 0 -> 1
- net S$45: track 23.0 -> 0.00 mm
- net S$23: track 2060.7 -> 2046.5 mm
- net S$42: track 5.41 -> 0.00 mm
- net S$43: track 4.00 -> 0.00 mm
- net S$25: track 1.23 -> 0.00 mm
- added copper zone on layer 1, net +24
- added copper zone on layer 1, net GND
Other:
- outline, holes or cut-outs redrawn

Commit message: BCN3D Electronics REV.E tested and manufactured
Parts:
- removed E$11, E$8, E$9: (no value), mk2i:HOT_DONT_TOUCH_LG
- removed E$12, E$7: (no value), mk2i:HOT_LG
- removed LED2: LED2, led:CHIPLED_0805
- removed NTC: 100K, SparkFun-Connectors:1X02
- removed R1K: (no value), resistor:R0805
- added CON: (no value), MarcEagleParts:MOLEX_MINIFIT-JR
- added E$3: (no value), MarcEagleParts:CE_BURNT_TAG
- added R1: (no value), resistor:R0805
- E$5: device MarcEagleParts:BCN3D_PRINTER_HUGE -> mk2i:HOT_LG
- E$6: device mk2i:HOT_LG -> mk2i:HOT_DONT_TOUCH_LG
- moved LED1 288.0 mm to (3.50, 147.5), turned to 180 degrees
- moved E$5 199.5 mm to (270.0, 55.0), flipped to the bottom
- moved E$13 55.0 mm to (60.0, 170.0), turned to 270 degrees
- moved E$6 53.9 mm to (63.0, 55.0), flipped to the bottom
- moved E$10 29.5 mm to (270.0, 170.0), turned to 270 degrees
- moved 100K-NTC 20.2 mm to (168.5, 105.0)
Routing:
- net R1: track 0.00 -> 16918.4 mm
- net R3: track 0.00 -> 16877.9 mm
- net R2: track 0.00 -> 16640.8 mm
- net R4: track 0.00 -> 16590.4 mm
- net S$4: track 3549.7 -> 26.2 mm
- net S$40: track 2114.6 -> 0.00 mm
- net S$12: track 2060.7 -> 0.00 mm
- net S$34: track 2060.2 -> 0.00 mm
- net S$23: track 2046.5 -> 0.00 mm
- net S$15: track 1875.3 -> 0.00 mm
- net S$26: track 1874.4 -> 0.00 mm
- net S$13: track 1874.0 -> 0.00 mm
- net S$8: track 1866.9 -> 0.00 mm
- net S$7: track 1866.9 -> 0.00 mm
- net S$37: track 1866.9 -> 0.00 mm
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- added copper zone on layer 1, net +24V
- added copper zone on layer 1, net HOTBED
- removed copper zone on layer 1, net +24
- removed copper zone on layer 1, net S$1
Other:
- board size 297 x 210 mm -> 305 x 198 mm
- board text added: "BCN3D Electronics BCN3D Technologies Fundacio CIM _______________________ Designed in Barcelona - 2014 Heated Platform - A4 Size 140 W output Power @ 24V Resistance between 3.8-4.2 Ohms"
- board text added: "REV_E"
- board text added: "THERM"
- board text removed: "Marc Cobler - REV_A"
- board text removed: "RepRapBCN - BCN3D Electronics __________________________ Designed in Barcelona - 2014 Heated Platform - A4 Size 120 W output Power @ 24V Resistance between 4.5-5 Ohms"
