File: MotherBoard/BCN3D electronics.sch (EAGLE design)
At the start: 86 parts, among them IC2 FT232RL, Q2 IRLS3034

Commit message: New File Tree and Updates
Connections:
- removed net 11111: ATMEGA2560.(OC2A/PCINT4)_PB4
- removed net N$156: ATMEGA2560.(OC5A)_PL3
- removed net N$157: ATMEGA2560.(OC5B)_PL4
- removed net N$158: ATMEGA2560.OC5C)_PL5
- net GND: no longer U$1.GND-SCREW
- net HOTEND2: now also ATMEGA2560.OC5C)_PL5
- net HOTEND3: now also ATMEGA2560.(OC2A/PCINT4)_PB4
- net LFAN2: now also ATMEGA2560.(OC5B)_PL4
- net LFAN3: now also ATMEGA2560.(OC5A)_PL3
Other:
- note added: "BCN3D - Barcelona 2014 Marc Cobler Cosmen www.fundaciocim.org"
- note added: "BCN3D electronics MotherBoard"
- note added: "Integrated electronics for controlled numeric Machines."
- note added: "USB"
- note removed: "BCN3D++ Mother Board"
- note removed: "Integrated 3D printer electronics for RepRap Machines."
- note removed: "RepRapBCN - Barcelona 2014 Marc Cobler Cosmen www.reprapbcn.com"
Changed lines of the file:
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@@
 <text x="246.38" y="271.78" size="2.54" layer="94">Extension Pin Header</text>
 <text x="132.08" y="259.08" size="1.9304" layer="97">4D Systems Display. Communication through serial.</text>
-<text x="93.98" y="340.36" size="2.54" layer="97">RepRapBCN - Barcelona 2014
+<text x="93.98" y="340.36" size="2.54" layer="97">BCN3D - Barcelona 2014
 Marc Cobler Cosmen
-www.reprapbcn.com</text>
+www.fundaciocim.org</text>
 <text x="66.04" y="325.12" size="2.54" layer="91">Design based on the Megatronics V3.0 and SAV mkI.
 Released under the Creative Commons Attribution Share-Alike 3.0 License</text>
-<text x="66.04" y="332.74" size="2.54" layer="91">Integrated 3D printer electronics for RepRap Machines. </text>
+<text x="66.04" y="332.74" size="2.54" layer="91">Integrated electronics for controlled numeric Machines. </text>
 <text x="370.84" y="360.68" size="2.54" layer="94">Stepper outputs</text>
 <wire x1="281.94" y1="368.3" x2="401.32" y2="368.3" width="0.6096" layer="94"/>
@@
 <wire x1="-60.96" y1="368.3" x2="-60.96" y2="309.88" width="0.6096" layer="94"/>
 <frame x1="-66.04" y1="71.12" x2="406.4" y2="373.38" columns="8" rows="5" layer="94"/>
-<text x="-12.7" y="330.2" size="2.54" layer="94">BCN3D++ Mother Board </text>
+<text x="-20.32" y="330.2" size="2.54" layer="94">BCN3D electronics MotherBoard </text>
 <text x="40.64" y="330.2" size="2.54" layer="94">A</text>
 <wire x1="129.54" y1="233.68" x2="228.6" y2="233.68" width="0.6096" layer="94"/>
@@
 <text x="299.72" y="134.62" size="1.778" layer="98">Dual smart Extruder config</text>
 <text x="332.74" y="134.62" size="1.778" layer="98">Dual Carriage Upgrade</text>
+<text x="-7.62" y="137.16" size="1.778" layer="98" rot="R90">Display</text>
+<text x="-7.62" y="121.92" size="1.778" layer="98" rot="R90">USB</text>
 </plain>
 <instances>
@@
 </segment>
 <segment>
-<pinref part="U$1" gate="G$1" pin="GND-SCREW"/>
-<wire x1="215.9" y1="358.14" x2="218.44" y2="358.14" width="0.1524" layer="91"/>
 <wire x1="218.44" y1="358.14" x2="218.44" y2="347.98" width="0.1524" layer="91"/>
-<pinref part="U$4" gate="G$1" pin="GND-SCREW"/>
+<pinref part="GND9" gate="1" pin="GND"/>
 <wire x1="218.44" y1="347.98" x2="218.44" y2="337.82" width="0.1524" layer="91"/>
 <wire x1="218.44" y1="337.82" x2="218.44" y2="327.66" width="0.1524" layer="91"/>
 <wire x1="218.44" y1="327.66" x2="218.44" y2="322.58" width="0.1524" layer="91"/>
-<wire x1="215.9" y1="327.66" x2="218.44" y2="327.66" width="0.1524" layer="91"/>
-<pinref part="U$3" gate="G$1" pin="GND-SCREW"/>
-<wire x1="215.9" y1="337.82" x2="218.44" y2="337.82" width="0.1524" layer="91"/>
 <pinref part="U$2" gate="G$1" pin="GND-SCREW"/>
 <wire x1="215.9" y1="347.98" x2="218.44" y2="347.98" width="0.1524" layer="91"/>
 <junction x="218.44" y="347.98"/>
+<pinref part="U$3" gate="G$1" pin="GND-SCREW"/>
+<wire x1="215.9" y1="337.82" x2="218.44" y2="337.82" width="0.1524" layer="91"/>
 <junction x="218.44" y="337.82"/>
+<pinref part="U$4" gate="G$1" pin="GND-SCREW"/>
+<wire x1="215.9" y1="327.66" x2="218.44" y2="327.66" width="0.1524" layer="91"/>
 <junction x="218.44" y="327.66"/>
-<pinref part="GND9" gate="1" pin="GND"/>
 </segment>
 <segment>
@@
 </segment>
 </net>
-<net name="N$156" class="0">
-<segment>
-<pinref part="ATMEGA2560" gate="A" pin="(OC5A)_PL3"/>
-<wire x1="104.14" y1="119.38" x2="124.46" y2="119.38" width="0.1524" layer="91"/>
-</segment>
-</net>
-<net name="N$157" class="0">
-<segment>
-<pinref part="ATMEGA2560" gate="A" pin="(OC5B)_PL4"/>
-<wire x1="104.14" y1="116.84" x2="124.46" y2="116.84" width="0.1524" layer="91"/>
-</segment>
-</net>
-<net name="N$158" class="0">
-<segment>
-<pinref part="ATMEGA2560" gate="A" pin="OC5C)_PL5"/>
-<wire x1="104.14" y1="114.3" x2="124.46" y2="114.3" width="0.1524" layer="91"/>
-</segment>
-</net>
 <net name="N$159" class="0">
 <segment>
@@
 <label x="347.98" y="144.78" size="1.778" layer="95"/>
 </segment>
+<segment>
+<pinref part="ATMEGA2560" gate="A" pin="(OC2A/PCINT4)_PB4"/>
+<wire x1="12.7" y1="182.88" x2="-5.08" y2="182.88" width="0.1524" layer="91"/>
+<label x="-2.54" y="182.88" size="1.778" layer="95"/>
+</segment>
 </net>
 <net name="LFAN0" class="0">
@@
 <label x="347.98" y="172.72" size="1.778" layer="95"/>
 </segment>
+<segment>
+<pinref part="ATMEGA2560" gate="A" pin="OC5C)_PL5"/>
+<wire x1="104.14" y1="114.3" x2="124.46" y2="114.3" width="0.1524" layer="91"/>
+<label x="109.22" y="114.3" size="1.778" layer="95"/>
+</segment>
 </net>
 <net name="LFAN2" class="0">
@@
 <label x="347.98" y="175.26" size="1.778" layer="95"/>
 </segment>
+<segment>
+<pinref part="ATMEGA2560" gate="A" pin="(OC5B)_PL4"/>
+<wire x1="104.14" y1="116.84" x2="124.46" y2="116.84" width="0.1524" layer="91"/>
+<label x="109.22" y="116.84" size="1.778" layer="95"/>
+</segment>
 </net>
 <net name="THERM2" class="0">
@@
 <wire x1="345.44" y1="147.32" x2="360.68" y2="147.32" width="0.1524" layer="91"/>
 <label x="347.98" y="147.32" size="1.778" layer="95"/>
+</segment>
+<segment>
+<pinref part="ATMEGA2560" gate="A" pin="(OC5A)_PL3"/>
+<wire x1="104.14" y1="119.38" x2="124.46" y2="119.38" width="0.1524" layer="91"/>
+<label x="109.22" y="119.38" size="1.778" layer="95"/>
 </segment>
 </net>
@@
 </segment>
 </net>
-<net name="11111" class="0">
-<segment>
-<pinref part="ATMEGA2560" gate="A" pin="(OC2A/PCINT4)_PB4"/>
-<wire x1="12.7" y1="182.88" x2="-5.08" y2="182.88" width="0.1524" layer="91"/>
-</segment>
-</net>

Commit message: Updates!
Rev_A Ready and firsts prototypes
Parts:
- removed PTC1: (no value), SAV MK-I:MICROBUILDER_PTC1206_L
- added F3: (no value), SAV MK-I:MICROBUILDER_PTC1206_L
- +24V, +24V1, ALVL, CARRIAGE0, CARRIAGE1, CARRIAGE2, CARRIAGE3, E0-AXIS, E1-AXIS, E2-AXIS, E3-AXIS, ENDSTOPS, FANS, FID1, FID2, FID3, HOTBED, ICSP, LCD, LOGO1, RGBLEDS, SD, THERM, U$1, U$2, U$3, U$4, X0-AXIS, X1-AXIS, X2-AXIS, X3-AXIS, Y0-AXIS, Y1-AXIS, Z-AXIS: OC_FARNELL (none) -> unknown
- +5V, 24V, GND, L2, L4: MF (none) -> MURATA; MPN (none) -> BLM31PG121SH1L; OC_FARNELL (none) -> 2443260
- ATMEGA2560: MF (none) -> ATMEL
- C1, C2: MF (none) -> AVX; MPN (none) -> 08055A220KAT2A; OC_FARNELL (none) -> 2332763
- C15, C20, C3, C4, C5, C6, C9: MF (none) -> AVX; MPN (none) -> 08055C104KAT2A; OC_FARNELL (none) -> 499687
- C21: MF (none) -> AVX; MPN (none) -> 06035C103JAT2A; OC_FARNELL (none) -> 1833871
- C7: MF (none) -> KEMET; MPN (none) -> C1206C475K5PACTU; OC_FARNELL (none) -> 1572637
- C8: MF (none) -> PANASONIC ELECTRONIC COMPONENTS; MPN (none) -> EEE1VA221UAP; OC_FARNELL (none) -> 2326175
- D1: MF (none) -> ON SEMICONDUCTOR; MPN (none) -> MBRS140T3G; OC_FARNELL (none) -> 9557237
- D3, D8: MF (none) -> PANASONIC ELECTRONIC COMPONENTS; MPN (none) -> DA22F2100L; OC_FARNELL (none) -> 2284096
- D9: MF (none) -> MULTICOMP; MPN (none) -> SS54; OC_FARNELL (none) -> 1861427
- F1: value PTCSMD -> IN_PTC; MF (none) -> SCHURTER; MPN (none) -> 3413.0329.22; OC_FARNELL (none) -> 1829472
- IC2: MF (none) -> FTDI
- L1: MF (none) -> BOURNS; MPN (none) -> SRR1260-101M; OC_FARNELL (none) -> 2396102
- LED2: MF (none) -> MULTICOMP; MPN (none) -> OVS-0803; OC_FARNELL (none) -> 1716765
- LM2595: MF (none) -> TEXAS INSTRUMENTS; MPN (none) -> LM2595S-5.0/NOPB; OC_FARNELL (none) -> 1469193
- PRW5, PWR24: MF (none) -> MULTICOMP; MPN (none) -> MCL-S270SRC; OC_FARNELL (none) -> 1581239
- Q2: MF (none) -> INTERNATIONAL RECTIFIER; MPN (none) -> IRLS3034PBF; OC_FARNELL (none) -> 1698309
- Q6, Q7, Q8: MF (none) -> NXP; MPN (none) -> BSH103,215; OC_FARNELL (none) -> 1081307
- R1: MF (none) -> MULTICOMP; MPN (none) -> MC0805S8F1004T5E; OC_FARNELL (none) -> 1646371
- R16, R19, R33, R34, R35, R36, R39: MF (none) -> BOURNS; MPN (none) -> CR0805-JW-102ELF; OC_FARNELL (none) -> 2008389
- R17, R37: MF (none) -> BOURNS; MPN (none) -> CR0805-JW-103ELF; OC_FARNELL (none) -> 2008390
- R2, R28, R38: MF (none) -> BOURNS; MPN (none) -> CR0805-FX-4701GLF; OC_FARNELL (none) -> 2008383
- RESET: MF (none) -> PANASONIC ELECTRONIC COMPONENTS; MPN (none) -> EVQPT9A15; OC_FARNELL (none) -> 2425618
- RXLED, TXLED: MF (none) -> WURTH ELEKTRONIK; MPN (none) -> 150060VS75000; OC_FARNELL (none) -> 2322073
- USB: MF (none) -> TE CONNECTIVITY / AMP; MPN (none) -> 1734035-1.; OC_FARNELL (none) -> 1654060
- Y1: MF (none) -> VISHAY DALE; MPN (none) -> XT49S 20M XT49S-20 B04 E2; OC_FARNELL (none) -> 1469646
Connections:
- net GND: now also U$1.GND-SCREW
- net N$5: now also F3.2; no longer PTC1.2
- net N$84: now also F3.1; no longer PTC1.1

Commit message: Updated files
Parts:
- removed USB: MINI-USB-SCHIELD, con-cypressindustries:MINI-USB-SCHIELD-32005-201
- added U$6: USB+SHIELD, SparkFun-Connectors:USB+SHIELD
- C7: value 4.7u -> 150UF; device rcl:C-EUC1206K -> MarcEagleParts:EEE-FK0J221P-CASE-D; MF KEMET -> (none); MPN C1206C475K5PACTU -> (none); OC_FARNELL 1572637 -> (none)
- D1: value MBRS140 -> (none); device MarcEagleParts:SHOTTKY-DIODESMBRS140 -> diode:SCHOTTKY-DIODESMC; MF ON SEMICONDUCTOR -> (none); MPN MBRS140T3G -> (none); OC_FARNELL 9557237 -> (none)
- LED2, RXLED, TXLED: device adafruit:LEDCHIP-LED0603 -> led:LEDCHIPLED_0805
Connections:
- removed net N$84: F3.1, USBG$1.1
- removed net USBSHIELD: L4.1, USBG$1.5, USBS.S1, USBS.S2, USBS.S3, USBS.S4
- new net N$23: F3.1, U$6.VBUS
- net +24V: now also C8.+; no longer C7.1
- net +5V: now also C7.1; no longer C8.+
- net N$22: now also L4.1, U$6.GND, U$6.S1, U$6.S2; no longer USBG$1.4
- net USBD+: now also U$6.D+; no longer USBG$1.3
- net USBD-: now also U$6.D-; no longer USBG$1.2
Other:
- moved on the sheet: C8, D1, D8, F3, L2, L4

Commit message: The new REV_B has been shipped to production
New MainBoard Design, new Stepper drivers and new Extruder Board.
We also added many new components and configurations
Parts:
- removed +24V: control, SparkFun-Connectors:M025MM
- removed +24V1: HEATED BED, SparkFun-Connectors:M025MM
- removed +5V, 24V, GND: PTR1TP12SQ, testpad:PTR1TP12SQ
- removed ALVL, THERM: (no value), pinhead:PINHD-1X2
- removed CARRIAGE0, CARRIAGE1, CARRIAGE2, CARRIAGE3, E0-AXIS, E1-AXIS, E2-AXIS, E3-AXIS, LCD, SD, X0-AXIS, X1-AXIS, X2-AXIS, X3-AXIS, Y0-AXIS, Y1-AXIS, Z-AXIS: (no value), MarcEagleParts:M06SIP
- removed ENDSTOPS: (no value), MarcEagleParts:PINCONNECTOR-7X3
- removed FANS: (no value), jumper:JP4QE
- removed HOTBED: M025MM, SparkFun-Connectors:M025MM
- removed L4: (no value), SAV MK-I:WUERTH-ELEKTRONIK_WE-CBF_1206W
- removed RESET: SWITCHSMD, SparkFun-Electromechanical:TAC_SWITCHSMD
- added ADC, SERIAL1: (no value), SparkFun-Connectors:M04PTH
- added C10: 100n, rcl:C-USC0805
- added C11: 0.1u, rcl:C-USC0805
- added C12, C13: 100u, rcl:CPOL-USUD-8X10
- added C14, C16: 10u, rcl:C-USC1210K
- added C17: 4.7u, adafruit:C-USC0805
- added C18: 10n, adafruit:C-USC0805
- added D2, D4, D5, D6, D7: MBRA140, SparkFun-DiscreteSemi:DIODESMA
- added E0, E1, X0, X1, Y0, Z: FFC_15V_90G_1MM, MarcEagleParts:FFC_15V_90G_1MM
- added HEATEDBED, SUPPLY: PC4WAY, MarcEagleParts:POWER_CONNECTOR_4WAY
- added HOTEND0, HOTEND1: FFC_20V_90G_1MM", MarcEagleParts:FFC_20V_90G_1MM"
- added HTST1: HTST_20V_SMD_POL, MarcEagleParts:HTST_20V_SMD_POL
- added IC3: LMV324MZ, linear:LMV324MZ
- added JP1: +5V, jumper:JP2Q
- added JP2: +24V, jumper:JP2Q
- added K1: G5L, relay:G5L
- added LED1, LED3: (no value), led:LEDCHIPLED_0805
- added Q1, Q3: MOSFET-N, MarcEagleParts:MOSFET-N
- added Q4, Q5, Q9: BC817, SparkFun-DiscreteSemi:TRANSISTOR_NPNMMBT2222A
- added R10, R13, R4, R5, R7: 10K, rcl:R-US_M0805
- added R11, R8: 5.6k, rcl:R-US_M0805
- added R12, R14, R15, R20, R21, R22, R6, R9: 1K, rcl:R-US_M0805
- added R18: 10K, pot:TRIM_US-3223J
- added R23, R24, R25: VARISTORCN0805, varistor:VARISTORCN0805
- added R3: 1K, rcl:R-US_R0805
- added RST: SPST_TACT-EVQQ2, adafruit:SPST_TACT-EVQQ2
- added S1: (no value), SparkFun-Electromechanical:SWITCH-SPDTPTH
- added STAT: Orange, adafruit:LEDCHIP-LED0805
- added TP1, TP10, TP11, TP12, TP13, TP14, TP15, TP16, TP17, TP18, TP2, TP3, TP4, TP5, TP6, TP7, TP8, TP9: TPB2,54, testpad:TPB2,54
- C21: value 10n -> 100n; device adafruit:C-USC0805K -> adafruit:C-USC0805
- D3: value MBR0520LT -> MBRA140; device diode:MBR0520LT -> SparkFun-DiscreteSemi:DIODESMA; MF PANASONIC ELECTRONIC COMPONENTS -> (none); MPN DA22F2100L -> (none); OC_FARNELL 2284096 -> (none)
- D9: value CGRM4004-G -> MBRA140; device diode:CGRM4004-G -> SparkFun-DiscreteSemi:DIODESMA; MF MULTICOMP -> (none); MPN SS54 -> (none); OC_FARNELL 1861427 -> (none)
- L2: value (none) -> 1800367 Ferrite Bead; device SAV MK-I:WUERTH-ELEKTRONIK_WE-CBF_1206W -> rcl:R-US_M0805; MF MURATA -> BOURNS; MPN BLM31PG121SH1L -> CR0805-JW-102ELF; OC_FARNELL 2443260 -> 2008389
- LED2: value HOTBED -> (none)
- Q2: value IRLS3034 -> MOSFET-N; device transistor-power:IRF3704S -> MarcEagleParts:MOSFET-N; MF INTERNATIONAL RECTIFIER -> (none); MPN IRLS3034PBF -> (none); OC_FARNELL 1698309 -> (none)
- R16: value 1K -> 4.7K; MPN CR0805-JW-102ELF -> CR0805-FX-4701GLF; OC_FARNELL 2008389 -> 2008383
- R17: value 10K -> 4.7K; MPN CR0805-JW-103ELF -> CR0805-FX-4701GLF; OC_FARNELL 2008390 -> 2008383
- R2: value 4.7K -> 5.6k; MPN CR0805-FX-4701GLF -> CR0805-JW-102ELF; OC_FARNELL 2008383 -> 2008389
- R38: value 4.7K -> 5.6K
Connections:
- net N$1 renamed XTAL_N
- net N$3 renamed XTAL_P
- net N$4 renamed OUT
- removed net AUTO_LEVEL: ALVL.1, ATMEGA2560.PK5_(ADC13/PCINT21), C9.1, R2.1
- removed net E-DIR: ATMEGA2560.PA1_(AD1), E0-AXIS.5, E1-AXIS.5, E2-AXIS.5, E3-AXIS.5
- removed net E-STEP: ATMEGA2560.PA0_(AD0), E0-AXIS.6, E1-AXIS.6, E2-AXIS.6, E3-AXIS.6
- removed net E2-!EN: ATMEGA2560.PA4_(AD4), E2-AXIS.4
- removed net E3-!EN: ATMEGA2560.PA5_(AD5), E3-AXIS.4
- removed net HOTEND2: ATMEGA2560.OC5C)_PL5, CARRIAGE2.2
- removed net HOTEND3: ATMEGA2560.(OC2A/PCINT4)_PB4, CARRIAGE3.2
- removed net LFAN2: ATMEGA2560.(OC5B)_PL4, CARRIAGE2.3
- removed net LFAN3: ATMEGA2560.(OC5A)_PL3, CARRIAGE3.3
- removed net N$129: ATMEGA2560.(RXD2)_PH0
- removed net N$130: ATMEGA2560.(TXD2)_PH1
- removed net N$131 (its old number): ATMEGA2560.(XCK2)_PH2
- removed net N$151: ATMEGA2560.PK6_(ADC14/PCINT22)
- removed net N$152: ATMEGA2560.PK7_(ADC15/PCINT23)
- removed net N$5: C21.1, F3.2, L2.2
- removed net N$83 (its old number): D8.A, L2.1
- removed net N$92: ATMEGA2560.PC1_(A9)
- removed net N$93: ATMEGA2560.PC2_(A10)
- removed net N$94: ATMEGA2560.PC3_(A11)
- removed net N$95: ATMEGA2560.PC4_(A12)
- removed net N$96: ATMEGA2560.PC5_(A13)
- removed net N$97: ATMEGA2560.PC6_(A14)
- removed net N$98: ATMEGA2560.PC7_(A15)
- removed net THERM0: ATMEGA2560.PK2_(ADC10/PCINT18), CARRIAGE0.1
- removed net THERM1: ATMEGA2560.PK1_(ADC9/PCINT17), CARRIAGE1.1
- removed net THERM2: ATMEGA2560.PK3_(ADC11/PCINT19), CARRIAGE2.1
- removed net THERM3: ATMEGA2560.PK4_(ADC12/PCINT20), CARRIAGE3.1
- removed net USBD+: IC2.USBDP, U$6.D+
- removed net USBD-: IC2.USBDM, U$6.D-
- removed net X-DIR: ATMEGA2560.PF2_(ADC2), X0-AXIS.5, X1-AXIS.5, X2-AXIS.5, X3-AXIS.5
- removed net X-STEP: ATMEGA2560.PF1_(ADC1), X0-AXIS.6, X1-AXIS.6, X2-AXIS.6, X3-AXIS.6
- removed net X2-!EN: ATMEGA2560.PF5_(ADC5/TMS), X2-AXIS.4
- removed net X2-STOP: ATMEGA2560.PJ4_(PCINT13), ENDSTOPS-5.1
- removed net X3-!EN: ATMEGA2560.PF6_(ADC6/TDO), X3-AXIS.4
- removed net X3-STOP: ATMEGA2560.PJ5_(PCINT14), ENDSTOPS-6.1
- removed net Y0-!EN: ATMEGA2560.(OC3B/INT4)_PE4, Y0-AXIS.4
- removed net Y0-STOP: ATMEGA2560.PJ2_(XCK3/PCINT11), ENDSTOPS-3.1
- removed net Y1-!EN: ATMEGA2560.(OC3C/INT5)_PE5, Y1-AXIS.4
- removed net Y1-STOP: ATMEGA2560.PJ3_(PCINT12), ENDSTOPS-4.1
- new net 24VBF: F1.1, K12.P
- new net ADC10: ADC.1, ATMEGA2560.PK2_(ADC10/PCINT18)
- new net ADC11: ADC.2, ATMEGA2560.PK3_(ADC11/PCINT19)
- new net ADC12: ADC.3, ATMEGA2560.PK4_(ADC12/PCINT20)
- new net ADC13: ADC.4, ATMEGA2560.PK5_(ADC13/PCINT21)
- new net ATLVL0: HOTEND0.20, IC3B.+IN, TP4.TP
- new net ATLVL1: HOTEND1.20, IC3C.+IN, TP5.TP
- new net E0-DIR: ATMEGA2560.PA7_(AD7), E0.6
- new net E0-STEP: ATMEGA2560.PA5_(AD5), E0.8
- new net E0-STOP: ATMEGA2560.PA4_(AD4), E0.11
- new net E1-DIR: ATMEGA2560.PF3_(ADC3), E1.6
- new net E1-STEP: ATMEGA2560.PF1_(ADC1), E1.8
- new net E1-STOP: ATMEGA2560.PF0_(ADC0), E1.11
- new net H0-STOP: ATMEGA2560.PA1_(AD1), IC3B.OUT
- new net H1-STOP: ATMEGA2560.PA0_(AD0), IC3C.OUT
- new net HOTBED: D3.A, HEATEDBED.4, Q1.D, R2.1, TP6.TP
- new net HOTEND0_THERM: ATMEGA2560.PK1_(ADC9/PCINT17), C9.1, HOTEND0.3, R16.1, TP12.TP
- new net HOTEND1_THERM: ATMEGA2560.PK0_(ADC8/PCINT16), C11.1, HOTEND1.3, R17.1, TP11.TP
- new net LMIN: C8.+, D2.C, LM2595.IN
- new net MLED: ATMEGA2560.PK6_(ADC14/PCINT22), IC3A.+IN
- new net N$100: D4.A, K11.2, Q9.C
- new net N$102: LED3.C, R11.2
- new net N$103: Q3.G, R12.1, R13.1
- new net N$107: Q5.B, R15.1
- new net N$108: C12.+, C13.+, C14.1, C16.1, K12.S, S1.P, SUPPLY.1, SUPPLY.3
- new net N$110: IC3B.-IN, IC3C.-IN, R18.S
- new net N$111: HTST1.8
- new net N$112: HTST1.9
- new net N$114: ATMEGA2560.PJ0_(RXD3/PCINT9)
- new net N$115: HTST1.10
- new net N$116: HTST1.16
- new net N$117: HTST1.17
- new net N$118: HTST1.18
- new net N$119: HTST1.19
- new net N$120: HTST1.20
- new net N$121: S1.O
- new net N$122: ATMEGA2560.PJ1_(TXD3/PCINT10)
- new net N$123: ATMEGA2560.(OC4C)_PH5
- new net N$124: ATMEGA2560.(OC2B)_PH6
- new net N$126: ATMEGA2560.PJ2_(XCK3/PCINT11)
- new net N$26: IC3A.-IN, IC3A.OUT, R3.2
- new net N$27: Q6.G, R20.1
- new net N$28: R3.1, STAT.A
- new net N$29: ATMEGA2560.PA2_(AD2)
- new net N$31: Q7.G, R21.1
- new net N$32: Q8.G, R22.1
- new net N$33: ATMEGA2560.PA3_(AD3)
- new net N$73: ATMEGA2560.PF5_(ADC5/TMS)
- new net N$74: ATMEGA2560.PF6_(ADC6/TDO)
- new net N$75: ATMEGA2560.PF7_(ADC7/TDI)
- new net N$90: Q4.B, R14.1
- new net N$99: Q2.G, R10.1, R9.1
- new net PWM_HOTEND0: ATMEGA2560.OC5C)_PL5, R9.2
- new net PWM_HOTEND1: ATMEGA2560.(OC4B)_PH4, R12.2
- new net PWM_LFAN0: ATMEGA2560.(OC5B)_PL4, R14.2
- new net PWM_LFAN1: ATMEGA2560.(OC4A)_PH3, R15.2
- new net RELAY: ATMEGA2560.(OC2A/PCINT4)_PB4, R19.2
- new net RX1: ATMEGA2560.(RXD1/INT2)_PD2, SERIAL1.3
- new net TX1: ATMEGA2560.(TXD1/INT3)_PD3, SERIAL1.4
- new net USBD+_P: IC2.USBDP, R23.1, U$6.D+
- new net USBD-_N: IC2.USBDM, R24.1, U$6.D-
- new net VBUS: L2.2, R25.1, U$6.VBUS
- new net VBUSAF: C17.1, C18.1, C21.1, F3.2, L2.1
- new net VCC2: D2.A, JP2.1, JP2.3, PWR24.A, RGBLEDS.1, S1.S
- new net X0-DIR: ATMEGA2560.PJ3_(PCINT12), X0.6
- new net X0-STEP: ATMEGA2560.PJ5_(PCINT14), X0.8
- new net X1-DIR: ATMEGA2560.(OC3A/AIN1)_PE3, X1.6
- new net X1-STEP: ATMEGA2560.(OC3C/INT5)_PE5, X1.8
- new net Y-!EN: ATMEGA2560.PC5_(A13), Y0.7
- new net Y-STOP: ATMEGA2560.PC7_(A15), Y0.11
- net !RESET: now also RST.P, RST.P1; no longer RESET.1, RESET.2
- net +24V: now also D5.C, D6.C, D7.C, E0.1, E0.3, E0.5, E1.1, E1.3, E1.5, HEATEDBED.1, HOTEND0.10, HOTEND0.12, HOTEND0.18, HOTEND0.19, HOTEND0.8, HOTEND1.10, HOTEND1.12, HOTEND1.18, HOTEND1.19, HOTEND1.8, HOTEND1.GND|1, LED1.A, LED3.A, TP2.TP, X0.1, X0.3, X0.5, X1.1, X1.3, X1.5, Y0.1, Y0.3, Y0.5, Z.1, Z.3, Z.5, Z.GND@1; no longer 24V.TP, C8.+, CARRIAGE0.6, CARRIAGE1.6, CARRIAGE2.6, CARRIAGE3.6, E0-AXIS.1, E1-AXIS.1, E2-AXIS.1, E3-AXIS.1, FANS-1.1, FANS-2.1, HOTBED.1, LM2595.IN, PWR24.A, RGBLEDS.1, X0-AXIS.1, X1-AXIS.1, X2-AXIS.1, X3-AXIS.1, Y0-AXIS.1, Y1-AXIS.1, Z-AXIS.1
- net +5V: now also C10.1, D4.C, E0.12, E0.14, E1.12, E1.14, HOTEND0.1, HOTEND1.1, HTST1.1, HTST1.11, IC3P.V+, JP1.1, JP1.3, K11.1, R16.2, R17.2, R18.E, R4.1, R5.1, SERIAL1.1, TP3.TP, X0.12, X0.14, X1.12, X1.14, Y0.12, Y0.14, Z.12, Z.14; no longer +5V.TP, CARRIAGE0.4, CARRIAGE1.4, CARRIAGE2.4, CARRIAGE3.4, E0-AXIS.3, E1-AXIS.3, E2-AXIS.3, E3-AXIS.3, ENDSTOPS-1.3, ENDSTOPS-2.3, ENDSTOPS-3.3, ENDSTOPS-4.3, ENDSTOPS-5.3, ENDSTOPS-6.3, ENDSTOPS-7.3, FANS-3.1, FANS-4.1, LCD.5, R2.2, SD.6, X0-AXIS.3, X1-AXIS.3, X2-AXIS.3, X3-AXIS.3, Y0-AXIS.3, Y1-AXIS.3, Z-AXIS.3
- net B-PWM: now also R22.2; no longer Q8.G
- net BED_THERM: now also ATMEGA2560.PK7_(ADC15/PCINT23), HEATEDBED.3, TP18.TP; no longer ATMEGA2560.PK0_(ADC8/PCINT16), THERM.1
- net E0-!EN: now also ATMEGA2560.PA6_(AD6), E0.7; no longer ATMEGA2560.PA2_(AD2), E0-AXIS.4
- net E1-!EN: now also ATMEGA2560.PF2_(ADC2), E1.7; no longer ATMEGA2560.PA3_(AD3), E1-AXIS.4
- net G-PWM: now also R20.2; no longer Q6.G
- net GND: now also C10.2, C11.2, C12.-, C13.-, C14.2, C16.2, C17.2, C18.2, E0.10, E0.13, E0.15, E0.2, E0.4, E0.9, E0.GND@1, E0.GND@2, E1.10, E1.13, E1.15, E1.2, E1.4, E1.9, E1.GND@1, E1.GND@2, HEATEDBED.2, HOTEND0.11, HOTEND0.17, HOTEND0.2, HOTEND0.4, HOTEND0.7, HOTEND0.9, HOTEND0.GND@2, HOTEND0.GND|1, HOTEND1.11, HOTEND1.17, HOTEND1.2, HOTEND1.4, HOTEND1.7, HOTEND1.9, HOTEND1.GND@2, HTST1.12, HTST1.2, IC3P.V-, JP1.2, JP1.4, JP2.2, JP2.4, Q1.S, Q3.S, Q4.E, Q5.E, Q9.E, R10.2, R13.2, R18.A, R23.2, R24.2, R25.2, R7.2, RST.S, RST.S1, SERIAL1.2, STAT.C, SUPPLY.2, SUPPLY.4, TP1.TP, U$6.GND, U$6.S1, U$6.S2, X0.10, X0.13, X0.15, X0.2, X0.4, X0.9, X0.GND@1, X0.GND@2, X1.10, X1.13, X1.15, X1.2, X1.4, X1.9, X1.GND@1, X1.GND@2, Y0.10, Y0.13, Y0.15, Y0.2, Y0.4, Y0.9, Y0.GND@1, Y0.GND@2, Z.10, Z.13, Z.15, Z.2, Z.4, Z.9, Z.GND@2; no longer +24V.2, +24V1.2, ALVL.2, CARRIAGE0.5, CARRIAGE1.5, CARRIAGE2.5, CARRIAGE3.5, D9.A, E0-AXIS.2, E1-AXIS.2, E2-AXIS.2, E3-AXIS.2, ENDSTOPS-1.2, ENDSTOPS-2.2, ENDSTOPS-3.2, ENDSTOPS-4.2, ENDSTOPS-5.2, ENDSTOPS-6.2, ENDSTOPS-7.2, FANS-1.2, FANS-2.2, FANS-3.2, FANS-4.2, GND.TP, L4.2, LCD.4, R17.2, RESET.3, RESET.4, SD.5, THERM.2, X0-AXIS.2, X1-AXIS.2, X2-AXIS.2, X3-AXIS.2, Y0-AXIS.2, Y1-AXIS.2, Z-AXIS.2
- net HOTEND0: now also D5.A, HOTEND0.13, HOTEND0.14, HOTEND0.15, HOTEND0.16, Q2.D, R8.1, TP7.TP; no longer ATMEGA2560.(OC2B)_PH6, CARRIAGE0.2
- net HOTEND1: now also D6.A, HOTEND1.13, HOTEND1.14, HOTEND1.15, HOTEND1.16, Q3.D, R11.1, TP8.TP; no longer ATMEGA2560.(OC4B)_PH4, CARRIAGE1.2
- net LCDRESET: now also ATMEGA2560.(XCK2)_PH2, HTST1.15; no longer ATMEGA2560.(ICP1)_PD4, LCD.1
- net LCDRX: now also ATMEGA2560.(TXD2)_PH1, HTST1.14; no longer ATMEGA2560.(TXD1/INT3)_PD3, LCD.2
- net LCDTX: now also ATMEGA2560.(RXD2)_PH0, HTST1.13; no longer ATMEGA2560.(RXD1/INT2)_PD2, LCD.3
- net LFAN0: now also D7.A, HOTEND0.5, HOTEND0.6, Q4.C, TP9.TP; no longer ATMEGA2560.(OC4C)_PH5, CARRIAGE0.3
- net LFAN1: now also D9.A, HOTEND1.5, HOTEND1.6, Q5.C, TP10.TP; no longer ATMEGA2560.(OC4A)_PH3, CARRIAGE1.3
- net MISO: now also HTST1.4, TP16.TP; no longer SD.3
- net MOSI: now also HTST1.5, TP15.TP; no longer SD.2
- net N$113: now also ATMEGA2560.(OC0B)_PG5; no longer ATMEGA2560.(T3/INT6)_PE6
- net N$22: now also ATMEGA2560.(ICP1)_PD4; no longer L4.1, U$6.GND, U$6.S1, U$6.S2
- net N$23: now also D8.A; no longer U$6.VBUS
- net N$24: now also HTST1.7; no longer LCD.6
- net N$25: now also Q9.B, R19.1; no longer +24V.1, +24V1.1, F1.1
- net N$63: now also LED1.C, R2.2; no longer Q2.G, R16.1, R17.1
- net N$66: now also Q1.G, R6.1, R7.1; no longer D3.A, HOTBED.2, Q2.D, R19.1
- net N$69: now also ATMEGA2560.PF4_(ADC4/TCK); no longer LED2.C, R19.2
- net N$91: now also LED2.C, R8.2; no longer ATMEGA2560.PC0_(A8)
- net PWM_HOTBED: now also ATMEGA2560.(OC5A)_PL3, R6.2; no longer ATMEGA2560.(OC0B)_PG5, R16.2
- net R-PWM: now also R21.2; no longer Q7.G
- net RX0: now also TP13.TP
- net SCL: now also R4.2
- net SCLK: now also HTST1.3, TP17.TP; no longer SD.4
- net SDA: now also R5.2
- net SDSS: now also HTST1.6; no longer SD.1
- net TX0: now also TP14.TP
- net X0-!EN: now also ATMEGA2560.PJ4_(PCINT13), X0.7; no longer ATMEGA2560.PF3_(ADC3), X0-AXIS.4
- net X0-STOP: now also ATMEGA2560.PJ6_(PCINT15), X0.11; no longer ATMEGA2560.PJ0_(RXD3/PCINT9), ENDSTOPS-1.1
- net X1-!EN: now also ATMEGA2560.(OC3B/INT4)_PE4, X1.7; no longer ATMEGA2560.PF4_(ADC4/TCK), X1-AXIS.4
- net X1-STOP: now also ATMEGA2560.(T3/INT6)_PE6, X1.11; no longer ATMEGA2560.PJ1_(TXD3/PCINT10), ENDSTOPS-2.1
- net Y-DIR: now also ATMEGA2560.PC4_(A12), Y0.6; no longer ATMEGA2560.(OC3A/AIN1)_PE3, Y0-AXIS.5, Y1-AXIS.5
- net Y-STEP: now also ATMEGA2560.PC6_(A14), Y0.8; no longer ATMEGA2560.PF7_(ADC7/TDI), Y0-AXIS.6, Y1-AXIS.6
- net Z-!EN: now also ATMEGA2560.PC1_(A9), Z.7; no longer ATMEGA2560.PF0_(ADC0), Z-AXIS.4
- net Z-DIR: now also ATMEGA2560.PC0_(A8), Z.6; no longer ATMEGA2560.PA7_(AD7), Z-AXIS.5
- net Z-STEP: now also ATMEGA2560.PC2_(A10), Z.8; no longer ATMEGA2560.PA6_(AD6), Z-AXIS.6
- net Z-STOP: now also ATMEGA2560.PC3_(A11), Z.11; no longer ATMEGA2560.PJ6_(PCINT15), ENDSTOPS-7.1
Other:
- note added: "Analog RGB LED strip - 3 PWM outputs needed"
- note added: "Autoleveling"
- note added: "B"
- note added: "BCN3D - Barcelona 2014 Marc Cobler Cosmen www.reprapbcn.com www.fundaciocim.org"
- note added: "VCC2 (24V) it's only for the DC/DC Converter, the cooler fan and the LED's"
- note removed: "A"
- note removed: "Analog RGB LED strip - 3 PWM outputs needed Normally strips go to 12V but we have 24V in our board"
- note removed: "Auto Leveling"
- note removed: "BCN3D - Barcelona 2014 Marc Cobler Cosmen www.fundaciocim.org"
- note removed: "Dual Carriage Upgrade"
- note removed: "Dual carriage Upgrade"
- note removed: "Endstops"
- moved on the sheet: ATMEGA2560, C1, C15, C2, C20, C21, C3, C4, C5, C6, C7, C8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

Commit message: BCN3D Electronics REV.E tested and manufactured
Parts:
- removed HTST1: HTST_20V_SMD_POL, MarcEagleParts:HTST_20V_SMD_POL
- removed PRW5: Red, adafruit:LEDCHIP-LED0805
- removed RST: SPST_TACT-EVQQ2, adafruit:SPST_TACT-EVQQ2
- removed S1: (no value), SparkFun-Electromechanical:SWITCH-SPDTPTH
- removed SERIAL1: (no value), SparkFun-Connectors:M04PTH
- removed TP14, TP18, TP6: TPB2,54, testpad:TPB2,54
- removed U$1, U$2, U$3, U$4: SANGUINOLOLU_PLATED-SCREW, SAV MK-I:SANGUINOLOLU_PLATED-SCREW
- added C19: 100n, rcl:C-USC0805
- added C22, C23: 0.1u, rcl:C-USC0805
- added C24: 100n, adafruit:C-USC0805
- added C25: 10n, rcl:C-USC0805
- added D10: MBR0520LT, diode:MBR0520LT
- added I2C, LEDS1, UART1: (no value), SparkFun-Connectors:M04PTH
- added IC1: LM358D, linear:LM358D
- added L10, L11, L12, L13, L14, L15, L16, L17, L18, L19, L20, L21, L3, L4, L5, L6, L7, L8, L9: (no value), EagleLibrary_Wuerth_Elektronik_eiSos_V6_20140807:WE-CBF_0805
- added LCD, SD: (no value), pinhead:PINHD-1X6
- added PWR5: Blue, led:LEDCHIPLED_0805
- added R26, R29: 4.7K, rcl:R-US_M0805
- added R27, R30, R43, R45, R46, R47: 1K, rcl:R-US_M0805
- added R31, R40, R42: 10K, rcl:R-US_M0805
- added R32: 330, adafruit:R-US_M0805
- added R41: 20K, rcl:R-US_M0805
- added R44: 100K, rcl:R-US_M0805
- added RESET: SPST, adafruit:SPST_TACT-EVQQ2
- added RSHUNT: 10m, SparkFun-Resistors:RESISTOR2512
- added SH1: SHORTT5, shorts:SHORTT5
- added SJ1: (no value), jumper:SJ
- added TP19, TP20, TP21, TP22, TP23, TP24, TP25, TP26, TP27, TP28, TP29, TP30, TP31, TP32, TP33, TP34, TP35, TP36, TP37, TP38: TPB2,54, testpad:TPB2,54
- added U1: INA169, SparkFun-AnalogIC:INA169
- added VCC2: (no value), jumper:JP1E
- +24V: value +24V -> (none); OC_FARNELL (none) -> unknown
- +5V: value +5V -> (none); OC_FARNELL (none) -> unknown
- ADC, E0, E1, TP1, TP10, TP11, TP12, TP13, TP15, TP16, TP17, TP2, TP3, TP4, TP5, TP7, TP8, TP9, X0, X1, Y0, Z: OC_FARNELL (none) -> unknown
- C11, C15, C9: value 0.1u -> 10u
- C12, C13: MF (none) -> PANASONIC ELECTRONIC COMPONENTS; MPN (none) -> EEEFC1V101AP; OC_FARNELL (none) -> 1244377
- C14, C16: MF (none) -> MURATA; MPN (none) -> GRM32ER7YA106KA12L; OC_FARNELL (none) -> 1735537
- C18: MPN 06035C103JAT2A -> 08055C103KAT2A; OC_FARNELL 1833871 -> 499225
- C21: MPN 06035C103JAT2A -> 08055C104KAT2A; OC_FARNELL 1833871 -> 499687
- C7: MF (none) -> PANASONIC ELECTRONIC COMPONENTS; MPN (none) -> EEEFP1A151AP; OC_FARNELL (none) -> 1539463
- D1: MF (none) -> ON SEMICONDUCTOR; MPN (none) -> MBRS340T3G; OC_FARNELL (none) -> 9557377
- D2, D3, D4, D5, D6, D7, D9: MF (none) -> DIODES INC.; MPN (none) -> B140-13-F; OC_FARNELL (none) -> 1843670
- HEATEDBED, SUPPLY: MF (none) -> MOLEX; MPN (none) -> 39303045; OC_FARNELL (none) -> 9963553
- HOTEND0, HOTEND1: value FFC_20V_90G_1MM" -> FFC_20V_90G_1MM3; device MarcEagleParts:FFC_20V_90G_1MM" -> MarcEagleParts:FFC_20V_90G_1MM3; OC_FARNELL (none) -> unknown
- IC3: value LMV324MZ -> LM311D; device linear:LMV324MZ -> linear:LM311D
- K1: MF (none) -> OMRON ELECTRONIC COMPONENTS; MPN (none) -> G5LA-1 5DC; OC_FARNELL (none) -> 1455502
- L2: value 1800367 Ferrite Bead -> (none); device rcl:R-US_M0805 -> EagleLibrary_Wuerth_Elektronik_eiSos_V6_20140807:WE-CBF_0805; MF BOURNS -> (none); MPN CR0805-JW-102ELF -> (none); OC_FARNELL 2008389 -> unknown
- LED1, LED2, LED3: value (none) -> Blue
- LM2595: device linear:LM2596S -> MarcEagleParts:LM2595
- PWR24: value Red -> Blue; device adafruit:LEDCHIP-LED0805 -> led:LEDCHIPLED_0805; MPN MCL-S270SRC -> OVS-0803; OC_FARNELL 1581239 -> 1716765
- Q1, Q2, Q3: value MOSFET-N -> MOSFET-NSOIC8; device MarcEagleParts:MOSFET-N -> MarcEagleParts:MOSFET-NSOIC8; MF (none) -> INTERNATIONAL RECTIFIER; MPN (none) -> IRF8736PBF; OC_FARNELL (none) -> 1551903
- Q4, Q5, Q9: value BC817 -> MMBT2222A; MF (none) -> NXP; MPN (none) -> BC817-40; OC_FARNELL (none) -> 1081225
- R1: value 1M -> 10K; device resistor:R-US_R0805 -> rcl:R-US_M0805; MF MULTICOMP -> BOURNS; MPN MC0805S8F1004T5E -> CR0805-JW-102ELF; OC_FARNELL 1646371 -> 2008389
- R18: device pot:TRIM_US-3223J -> rcl:R-US_M0805; MF (none) -> BOURNS; MPN (none) -> CR0805-JW-102ELF; OC_FARNELL (none) -> 2008389
- R23, R24, R25: MF (none) -> LITTELFUSE; MPN (none) -> V5.5MLA0805LH; OC_FARNELL (none) -> 1057218
- R4, R5: value 10K -> 4.7k
- RXLED, TXLED: MPN 150060VS75000 -> 150080VS75000; OC_FARNELL 2322073 -> 2322081
- STAT: MF MULTICOMP -> KINGBRIGHT; MPN MCL-S270SRC -> KP-2012SECK; OC_FARNELL 1581239 -> 2290332
- U$6: MF (none) -> MOLEX; MPN (none) -> 67068-8000; OC_FARNELL (none) -> 1463095
- Y1: MF VISHAY DALE -> TXC; MPN XT49S 20M XT49S-20 B04 E2 -> 9B-16.000MAAJ-B; OC_FARNELL 1469646 -> 1842216
- renumbered JP1 to +5V, JP2 to +24V
Connections:
- removed net ATLVL0: HOTEND0.20, IC3B.+IN, TP4.TP
- removed net ATLVL1: HOTEND1.20, IC3C.+IN, TP5.TP
- removed net H0-STOP: ATMEGA2560.PA1_(AD1), IC3B.OUT
- removed net H1-STOP: ATMEGA2560.PA0_(AD0), IC3C.OUT
- removed net N$108: C12.+, C13.+, C14.1, C16.1, K12.S, S1.P, SUPPLY.1, SUPPLY.3
- removed net N$110: IC3B.-IN, IC3C.-IN, R18.S
- removed net N$111: HTST1.8
- removed net N$112: HTST1.9
- removed net N$115: HTST1.10
- removed net N$116: HTST1.16
- removed net N$117: HTST1.17
- removed net N$118: HTST1.18
- removed net N$119: HTST1.19
- removed net N$120: HTST1.20
- removed net N$121: S1.O
- removed net N$124: ATMEGA2560.(OC2B)_PH6
- removed net N$146: ATMEGA2560.PL6
- removed net N$25: Q9.B, R19.1
- removed net RX0: ATMEGA2560.(RXD0/PCINT8)_PE0, R35.1, TP13.TP
- removed net TX0: ATMEGA2560.(TXD0)_PE1, R36.1, TP14.TP
- removed net VBUSAF: C17.1, C18.1, C21.1, F3.2, L2.1
- new net 24VINA: K12.P, RSHUNT.1, U1.VIN+
- new net BED_THERM_CON: HEATEDBED.3, R45.1
- new net EARTH: L21.2, U$6.S1, U$6.S2
- new net GUARD: C1.2, C2.2, SH1.P$2
- new net HOTEND0_THERM_CON: HOTEND0.3, R46.1
- new net HOTEND1_THERM_CON: HOTEND1.3, R47.1
- new net INA_OUT: IC3.-IN, R41.2, U1.OUT
- new net N$1: C19.1, IC2.!DTR
- new net N$34: L13.1, X0.7
- new net N$35: L14.1, X0.9
- new net N$36: L18.1, Y0.6
- new net N$37: L19.1, Y0.7
- new net N$39: L20.1, Y0.9
- new net N$4: ATMEGA2560.(XCK2)_PH2
- new net N$40: L15.1, X1.6
- new net N$41: L16.1, X1.7
- new net N$42: L17.1, X1.9
- new net N$43: E0.6, L6.2
- new net N$44: E0.7, L7.2
- new net N$45: E0.9, L8.2
- new net N$47: ATMEGA2560.PC2_(A10)
- new net N$48: F3.2, L2.1
- new net N$49: IC3.+IN, R1.2, R42.1, R44.1
- new net N$5: L12.1, X0.6
- new net N$54: L3.1, Z.6
- new net N$55: L4.1, Z.7
- new net N$56: L5.1, Z.9
- new net N$57: E1.9, L11.1
- new net N$58: E1.7, L10.1
- new net N$59: E1.6, L9.1
- new net RELAYINA: IC3.OUT, Q9.B, R19.1, R43.2, R44.2, SJ1.1, SJ1.2
- new net SUPPLY: C12.+, C13.+, C14.1, C16.1, K12.S, LEDS1.1, PWR24.A, RGBLEDS.1, SUPPLY.1, SUPPLY.3, TP2.TP, VCC2.1
- new net UART_N: ATMEGA2560.(TXD0)_PE1, R36.1
- new net UART_P: ATMEGA2560.(RXD0/PCINT8)_PE0, R35.1
- new net Z0-ENDSTOP: HOTEND0.20, R26.1, R27.1
- new net Z0-STOP: ATMEGA2560.PC3_(A11), C22.1, R27.2
- new net Z1-ENDSTOP: HOTEND1.20, R29.1, R30.1
- new net Z1-STOP: ATMEGA2560.PL6, C23.1, R30.2
- net !RESET: now also C19.2, C25.1, D10.A, R32.1; no longer RST.P, RST.P1
- net +24V: now also Y0.GND@2; no longer HOTEND1.GND|1, TP2.TP, Z.GND@1
- net +5V: now also +24V.1, +24V.3, C17.1, C18.1, C21.1, C24.1, D10.C, I2C.1, IC1P.V+, IC3.V+, LCD.1, PWR5.A, R1.1, R26.2, R29.2, R43.1, SD.6, U1.V+, UART1.1; no longer +5V.1, +5V.3, HTST1.1, HTST1.11, IC3P.V+, PRW5.A, R18.E, SERIAL1.1
- net 24VBF: now also RSHUNT.2, U1.VIN-; no longer K12.P
- net BED_THERM: now also R45.2, TP13.TP; no longer HEATEDBED.3, TP18.TP
- net E0-!EN: now also L7.1, TP34.TP; no longer E0.7
- net E0-DIR: now also ATMEGA2560.PA5_(AD5), L8.1, TP33.TP; no longer ATMEGA2560.PA7_(AD7), E0.6
- net E0-STEP: now also ATMEGA2560.PA7_(AD7), L6.1, TP35.TP; no longer ATMEGA2560.PA5_(AD5), E0.8
- net E1-!EN: now also L10.2, TP31.TP; no longer E1.7
- net E1-DIR: now also ATMEGA2560.PF1_(ADC1), L11.2, TP32.TP; no longer ATMEGA2560.PF3_(ADC3), E1.6
- net E1-STEP: now also ATMEGA2560.PF3_(ADC3), L9.2, TP30.TP; no longer ATMEGA2560.PF1_(ADC1), E1.8
- net GND: now also C22.2, C23.2, C24.2, C25.2, E0.8, E1.8, HOTEND0.GND@1, HOTEND1.GND@1, I2C.2, IC1P.V-, IC3.GND, IC3.V-, L21.1, LCD.4, LCD.6, R18.2, R31.2, R40.2, R41.1, R42.2, RESET.P, RESET.P1, SD.1, SH1.P$1, U1.GND, UART1.2, X0.8, X1.8, Y0.8, Z.8, Z.GND@1; no longer C1.2, C2.2, E0.9, E1.9, HOTEND0.GND|1, HTST1.12, HTST1.2, IC3P.V-, R18.A, RST.S, RST.S1, SERIAL1.2, U$1.GND-SCREW, U$2.GND-SCREW, U$3.GND-SCREW, U$4.GND-SCREW, U$6.S1, U$6.S2, X0.9, X1.9, Y0.9, Y0.GND@2, Z.9
- net HOTBED: no longer TP6.TP
- net HOTEND0_THERM: now also R46.2; no longer HOTEND0.3
- net HOTEND1_THERM: now also R47.2; no longer HOTEND1.3
- net LCDRESET: now also ATMEGA2560.(OC2B)_PH6, LCD.5, TP4.TP; no longer ATMEGA2560.(XCK2)_PH2, HTST1.15
- net LCDRX: now also LCD.3, TP5.TP; no longer HTST1.14
- net LCDTX: now also LCD.2, TP15.TP; no longer HTST1.13
- net MISO: now also SD.2, TP20.TP; no longer HTST1.4, TP16.TP
- net MLED: now also IC1A.+IN; no longer IC3A.+IN
- net MOSI: now also SD.4, TP17.TP; no longer HTST1.5, TP15.TP
- net N$10: now also LEDS1.3
- net N$11: now also LEDS1.4
- net N$13: now also R32.2, RESET.S, RESET.S1; no longer IC2.!DTR
- net N$162: now also PWR5.C; no longer PRW5.C
- net N$23: now also L2.2; no longer F3.1
- net N$24: now also ATMEGA2560.PA0_(AD0); no longer HTST1.7
- net N$26: now also IC1A.-IN, IC1A.OUT; no longer IC3A.-IN, IC3A.OUT
- net N$27: now also R18.1
- net N$29: now also ATMEGA2560.PC0_(A8); no longer ATMEGA2560.PA2_(AD2)
- net N$31: now also R31.1
- net N$32: now also R40.1
- net N$33: now also ATMEGA2560.PC1_(A9); no longer ATMEGA2560.PA3_(AD3)
- net N$9: now also LEDS1.2
- net RX1: now also UART1.3; no longer SERIAL1.3
- net SCL: now also I2C.3
- net SCLK: now also SD.3, TP19.TP; no longer HTST1.3, TP17.TP
- net SDA: now also I2C.4
- net SDSS: now also SD.5, TP16.TP; no longer HTST1.6
- net TX1: now also UART1.4; no longer SERIAL1.4
- net VBUS: now also F3.1; no longer L2.2
- net VCC2: now also +5V.1, +5V.3, VCC2.2; no longer +24V.1, +24V.3, PWR24.A, RGBLEDS.1, S1.S
- net X0-!EN: now also L13.2, TP22.TP; no longer X0.7
- net X0-DIR: now also ATMEGA2560.PJ5_(PCINT14), L14.2, TP23.TP; no longer ATMEGA2560.PJ3_(PCINT12), X0.6
- net X0-STEP: now also ATMEGA2560.PJ3_(PCINT12), L12.2, TP21.TP; no longer ATMEGA2560.PJ5_(PCINT14), X0.8
- net X1-!EN: now also L16.2, TP25.TP; no longer X1.7
- net X1-DIR: now also ATMEGA2560.(OC3C/INT5)_PE5, L17.2, TP26.TP; no longer ATMEGA2560.(OC3A/AIN1)_PE3, X1.6
- net X1-STEP: now also ATMEGA2560.(OC3A/AIN1)_PE3, L15.2, TP24.TP; no longer ATMEGA2560.(OC3C/INT5)_PE5, X1.8
- net XTAL_N: no longer R1.2
- net XTAL_P: no longer R1.1
- net Y-!EN: now also ATMEGA2560.PC6_(A14), L19.2, TP28.TP; no longer ATMEGA2560.PC5_(A13), Y0.7
- net Y-DIR: now also ATMEGA2560.PC5_(A13), L20.2, TP29.TP; no longer ATMEGA2560.PC4_(A12), Y0.6
- net Y-STEP: now also ATMEGA2560.PC7_(A15), L18.2, TP27.TP; no longer ATMEGA2560.PC6_(A14), Y0.8
- net Y-STOP: now also ATMEGA2560.PC4_(A12); no longer ATMEGA2560.PC7_(A15)
- net Z-!EN: now also ATMEGA2560.PA2_(AD2), L4.2, TP37.TP; no longer ATMEGA2560.PC1_(A9), Z.7
- net Z-DIR: now also ATMEGA2560.PA1_(AD1), L5.2, TP36.TP; no longer ATMEGA2560.PC0_(A8), Z.6
- net Z-STEP: now also ATMEGA2560.PA3_(AD3), L3.2, TP38.TP; no longer ATMEGA2560.PC2_(A10), Z.8
- net Z-STOP: no longer ATMEGA2560.PC3_(A11)
Other:
- note added: "Analog RGB LED strip - 4 PWM outputs needed"
- note added: "BCN3D - Barcelona 2014 Marc Cobler Cosmen www.bcn3dtechnologies.com www.fundaciocim.org"
- note added: "BCN3D electronics MainBoard"
- note added: "CSM"
- note added: "CSM - Current Shunt Monitor"
- note added: "E"
- note added: "INA169 monitors current on the high side and acts on the relay. 0.2 Volt per Amp"
- note added: "VCC2 (24V) it's only for the DC/DC Converter and the LED's"
- note added: "Z-Endstops"
- note removed: "Analog RGB LED strip - 3 PWM outputs needed"
- note removed: "Autoleveling"
- note removed: "B"
- note removed: "BCN3D - Barcelona 2014 Marc Cobler Cosmen www.reprapbcn.com www.fundaciocim.org"
- note removed: "BCN3D electronics MotherBoard"
- note removed: "VCC2 (24V) it's only for the DC/DC Converter, the cooler fan and the LED's"
- moved on the sheet: ADC, C10, E0, F1, F3, Q6, Q7, Q8, R1, R14, R16, R17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
